Commit message: 4 legs

File: models/crab_leg.xacro (robot description, xacro)
@@ -41,4 +41,6 @@
     		<axis xyz="0 0 -1" />
     		<limit lower="${joint_lower_limit}" upper="${joint_upper_limit}" effort="${joint_effort}" velocity="${joint_velocity}" />
+				<limit lower="-1.0"
+							 upper="1.0"/>
   	</joint>
   	<link name="coxa_${side}${num}">

File: models/crab_model.xacro (robot description, xacro)
@@ -70,6 +70,6 @@
     </gazebo>
 <!-- Joint properties -->
-    <xacro:property name="joint_lower_limit" value="-${1.5}" />
-    <xacro:property name="joint_upper_limit" value="${1.5}" />
+    <xacro:property name="joint_lower_limit" value="-${0.8}" />
+    <xacro:property name="joint_upper_limit" value="${0.8}" />
     <xacro:property name="joint_effort" value="10000" />
     <xacro:property name="joint_velocity" value="100" />
