Commit message: Changed colour robot

File: models/crab_model.xacro (robot description, xacro)
@@ -38,5 +38,7 @@
     <gazebo reference="base_link">
         <selfCollide>true</selfCollide>
-        <material>Gazebo/Grey</material>
+        <material name="orange">
+          <color rgba="${255/255} ${108/255} ${10/255} 1.0"/>
+        </material>
     </gazebo>
     <link name="thorax">
@@ -80,5 +82,5 @@
     <gazebo reference="thorax">
         <selfCollide>true</selfCollide>
-        <material>Gazebo/Grey</material>
+        <material>Gazebo/Orange</material>
     </gazebo>
     <link name="leg_center_${side}${num}">

Commit message: Computed inertia from the thorax

File: models/crab_model.xacro (robot description, xacro)
@@ -102,9 +102,9 @@
         <inertial>
             <origin xyz="0 0 0" rpy="0 0 0"/>
-            <mass value="0.02"/>
-            <inertia
-                ixx="0.0001" ixy="0.0" ixz="0.0"
-                iyy="0.0001" iyz="0.0"
-                izz="0.0001"/>
+            <mass value="0.02"/> <!-- The mass has to be recomputed -->
+            <inertia
+                ixx="0.011935/10000" ixy="0.0" ixz="-0.000021/10000"
+                iyy="0.022562/10000" iyz="-0.000001/10000"
+                izz="0.026533/10000"/>
         </inertial>
     </link>

Commit message: Computed inertia of coxa joint

File: models/crab_model.xacro (robot description, xacro)
@@ -38,7 +38,5 @@
     <gazebo reference="base_link">
         <selfCollide>true</selfCollide>
-        <material name="orange">
-          <color rgba="${255/255} ${108/255} ${10/255} 1.0"/>
-        </material>
+        <material>Gazebo/Grey</material>
     </gazebo>
     <link name="thorax">
@@ -62,7 +60,7 @@
             <mass value="0.02"/>
             <inertia
-                ixx="0.0001" ixy="0.0" ixz="0.0"
-                iyy="0.0001" iyz="0.0"
-                izz="0.0001"/>
+              ixx="0.011935/10000" ixy="0.0" ixz="-0.000021/10000"
+              iyy="0.022562/10000" iyz="-0.000001/10000"
+              izz="0.026533/10000"/>
         </inertial>
     </link>
@@ -140,7 +138,7 @@
             <mass value="0.02"/>
             <inertia
-                ixx="0.0001" ixy="0.0" ixz="0.0"
-                iyy="0.0001" iyz="0.0"
-                izz="0.0001"/>
+                ixx="0.00138/10000" ixy="0.000093/10000" ixz="-0.000177/10000"
+                iyy="0.001442/10000" iyz="0.00003/10000"
+                izz="0.001371/10000"/>
         </inertial>
     </link>

Commit message: Transmisions in xacro

File: models/crab_model.xacro (robot description, xacro)
@@ -31,4 +31,8 @@
         </inertial>
     </link>
+    <gazebo reference="base_link">
+        <selfCollide>true</selfCollide>
+        <material>Gazebo/Grey</material>
+    </gazebo>
     <joint name="base_joint" type="fixed">
         <parent link="base_link" />
@@ -36,8 +40,4 @@
         <origin xyz="0 0 0" rpy="0 0 0" />
     </joint>
-    <gazebo reference="base_link">
-        <selfCollide>true</selfCollide>
-        <material>Gazebo/Grey</material>
-    </gazebo>
     <link name="thorax">
         <collision>
@@ -65,4 +65,8 @@
         </inertial>
     </link>
+    <gazebo reference="thorax">
+        <selfCollide>true</selfCollide>
+        <material>Gazebo/Grey</material>
+    </gazebo>
 <!-- Joint properties -->
     <xacro:property name="joint_lower_limit" value="-${1.5}" />
@@ -78,8 +82,4 @@
         <child link="leg_center_${side}${num}" />
     </joint>
-    <gazebo reference="thorax">
-        <selfCollide>true</selfCollide>
-        <material>Gazebo/Grey</material>
-    </gazebo>
     <link name="leg_center_${side}${num}">
         <collision>
@@ -118,4 +118,12 @@
         <limit lower="${joint_lower_limit}" upper="${joint_upper_limit}" effort="${joint_effort}" velocity="${joint_velocity}" />
     </joint>
+    <transmission name="tran_coxa_${side}${num}">
+      <type>transmission_interface/SimpleTransmission</type>
+      <joint name="coxa_joint_${side}${num}"> <hardwareInterface>EffortJointInterface</hardwareInterface> 	</joint>
+      <actuator name="motor_coxa_${side}${num}">
+        <hardwareInterface>EffortJointInterface</hardwareInterface>
+        <mechanicalReduction>1</mechanicalReduction>
+      </actuator>
+    </transmission>
     <link name="coxa_${side}${num}">
         <collision>
@@ -154,4 +162,12 @@
         <limit lower="${joint_lower_limit}" upper="${joint_upper_limit}" effort="${joint_effort}" velocity="${joint_velocity}" />
     </joint>
+    <transmission name="tran_femur_${side}${num}">
+      <type>transmission_interface/SimpleTransmission</type>
+      <joint name="femur_joint_${side}${num}"> <hardwareInterface>EffortJointInterface</hardwareInterface> 	</joint>
+      <actuator name="motor_femur_${side}${num}">
+        <hardwareInterface>EffortJointInterface</hardwareInterface>
+        <mechanicalReduction>1</mechanicalReduction>
+      </actuator>
+    </transmission>
     <link name="femur_${side}${num}">
         <collision>
@@ -190,4 +206,12 @@
         <limit lower="${joint_lower_limit}" upper="${joint_upper_limit}" effort="${joint_effort}" velocity="${joint_velocity}" />
     </joint>
+    <transmission name="tran_tibia_${side}${num}">
+      <type>transmission_interface/SimpleTransmission</type>
+      <joint name="tibia_joint_${side}${num}"> <hardwareInterface>EffortJointInterface</hardwareInterface> 	</joint>
+      <actuator name="motor_tibia_${side}${num}">
+        <hardwareInterface>EffortJointInterface</hardwareInterface>
+        <mechanicalReduction>1</mechanicalReduction>
+      </actuator>
+    </transmission>
     <link name="tibia_${side}${num}">
         <collision>
@@ -224,4 +248,12 @@
         <child link="tibia_foot_${side}${num}" />
     </joint>
+    <transmission name="tran_tibia_foot_${side}${num}">
+      <type>transmission_interface/SimpleTransmission</type>
+      <joint name="tibia_foot_joint_${side}${num}"> <hardwareInterface>EffortJointInterface</hardwareInterface> 	</joint>
+      <actuator name="motor_tibia_foot_${side}${num}">
+        <hardwareInterface>EffortJointInterface</hardwareInterface>
+        <mechanicalReduction>1</mechanicalReduction>
+      </actuator>
+    </transmission>
     <link name="tibia_foot_${side}${num}" />
     <gazebo reference="tibia_foot_${side}${num}">

Commit message: transmissions done in xacro

File: models/crab_model.xacro (robot description, xacro)
@@ -248,12 +248,4 @@
         <child link="tibia_foot_${side}${num}" />
     </joint>
-    <transmission name="tran_tibia_foot_${side}${num}">
-      <type>transmission_interface/SimpleTransmission</type>
-      <joint name="tibia_foot_joint_${side}${num}"> <hardwareInterface>EffortJointInterface</hardwareInterface> 	</joint>
-      <actuator name="motor_tibia_foot_${side}${num}">
-        <hardwareInterface>EffortJointInterface</hardwareInterface>
-        <mechanicalReduction>1</mechanicalReduction>
-      </actuator>
-    </transmission>
     <link name="tibia_foot_${side}${num}" />
     <gazebo reference="tibia_foot_${side}${num}">

Commit message: Simulation

File: models/crab_model.xacro (robot description, xacro)
@@ -58,5 +58,5 @@
         <inertial>
             <origin xyz="0 0 0" rpy="0 0 0"/>
-            <mass value="0.02"/>
+            <mass value="0.3"/>
             <inertia
                 ixx="0.0001" ixy="0.0" ixz="0.0"

Commit message: Updating branch with inertias and mass

File: models/crab_model.xacro (robot description, xacro)
@@ -40,8 +40,4 @@
         <origin xyz="0 0 0" rpy="0 0 0" />
     </joint>
-    <gazebo reference="base_link">
-        <selfCollide>true</selfCollide>
-        <material>Gazebo/Grey</material>
-    </gazebo>
     <link name="thorax">
         <collision>
@@ -62,5 +58,5 @@
         <inertial>
             <origin xyz="0 0 0" rpy="0 0 0"/>
-            <mass value="0.3"/>
+            <mass value="0.41"/>
             <inertia
               ixx="0.011935" ixy="0.0" ixz="-0.000021"
@@ -106,7 +102,7 @@
             <mass value="0.02"/> <!-- The mass has to be recomputed -->
             <inertia
-                ixx="0.011935" ixy="0.0" ixz="-0.000021"
-                iyy="0.022562" iyz="-0.000001"
-                izz="0.026533"/>
+                ixx="0.011935e-3" ixy="0.0" ixz="-0.000021e-3"
+                iyy="0.022562e-3" iyz="-0.000001e-3"
+                izz="0.026533e-3"/>
         </inertial>
     </link>
@@ -148,5 +144,5 @@
         <inertial>
             <origin xyz="0 0 0" rpy="0 0 0"/>
-            <mass value="0.02"/>
+            <mass value="0.0147"/>
             <inertia
                 ixx="0.00138" ixy="0.000093" ixz="-0.000177"
@@ -192,5 +188,5 @@
         <inertial>
             <origin xyz="0 0 0" rpy="0 0 0"/>
-            <mass value="0.02"/>
+            <mass value="0.032"/>
             <inertia
                 ixx="0.000012" ixy="0.0" ixz="0.0"
@@ -236,5 +232,5 @@
         <inertial>
             <origin xyz="0 0 0" rpy="0 0 0"/>
-            <mass value="0.02"/>
+            <mass value="0.008"/>
             <inertia
                 ixx="0.000317" ixy="-0.000054" ixz="-0.000061"

Commit message: Update

File: models/crab_model.xacro (robot description, xacro)
@@ -70,6 +70,6 @@
     </gazebo>
 <!-- Joint properties -->
-    <xacro:property name="joint_lower_limit" value="-${0.8}" />
-    <xacro:property name="joint_upper_limit" value="${0.8}" />
+    <xacro:property name="joint_lower_limit" value="-${1}" />
+    <xacro:property name="joint_upper_limit" value="${1}" />
     <xacro:property name="joint_effort" value="10000" />
     <xacro:property name="joint_velocity" value="100" />
